File: LedBandRadio_hw/LedBandRadio.kicad_pcb (KiCad board)
At the start: 2 copper layers, 60 x 79 mm, 99 parts, among them Q1 IRF8313, SW1 DIPx6, U1 USBLC6

Commit message: New +5V sch Still with 3-ch 12V LED control
Parts:
- removed D1, D2: BAT54WS, Diodes:SOD323
- added C44: 0.1u, Capacitors:CAP_0603, F.Cu at (190.8, 65.5)
- added C45: 0.1u, Capacitors:CAP_0603, F.Cu at (196.9, 57.8)
- added C46: 0.1u, Capacitors:CAP_0603, F.Cu at (196.9, 60.2)
- added C47: 0.1u, Capacitors:CAP_0603, F.Cu at (196.5, 65.5)
- added DA7: LP2951, SO_DIL_TSSOP:SO8_150MIL, F.Cu at (211.8, 60.5)
- added Q2: IRF8714, SO_DIL_TSSOP:SO8_150MIL, F.Cu at (189.9, 60.5)
- added R15: 10k, Resistors:RES_0603, F.Cu at (216.8, 57.8)
- C1, C6: value 10n -> 10u 16V; footprint Capacitors:CAP_0603 -> Capacitors:CAP_0805
- C10: value 0.22u -> 1u
- C11: value 1u -> 0.47u
- C21, C34: value 220pF -> 0.1u
- C23: value 10n -> 470pF
- C26: value 3.3pF -> 10n
- C28: value 10n -> 1u
- C8: value 1u -> 0.1u
- DA1: value MAX8546 -> LM3150; footprint SO_DIL_TSSOP:uMAX_uSOP10 -> SO_DIL_TSSOP:HTSSOP14
- F7: footprint Resistors:RES_0603_FUSE -> PCB:FuseShorted
- L1: footprint Inductors:13x14 -> Inductors:13x13
- Q1: value IRF8313 -> IRF8714
- R1: value 1M -> 100k
- R2: value 47k -> 2k
- R3: value 10R -> 75k
- R4: value 4.7k -> 10k
- R5: value 27k -> 12k
- R6: value 220R -> 1k
- moved XL3 75.6 mm to (236.2, 63.2), turned to 0 degrees
Connections:
- C1 pad 1: GND -> +BATT
- C1 pad 2: /SHLD -> GNDPWR
- C10 pad 2: Net-(C10-Pad2) -> GNDPWR
- C11 pad 1: GNDPWR -> /L1IN
- C21 pad 1: VCC -> +BATT
- C23 pad 1: VCC -> Net-(C23-Pad1)
- C23 pad 2: GND -> +5V
- C26 pad 1: VCC -> +3.3V
- C26 pad 2: GND -> Net-(C26-Pad2)
- C6 pad 1: GNDPWR -> +BATT
- C6 pad 2: Net-(C6-Pad2) -> GNDPWR
- C8 pad 1: GNDPWR -> Net-(C8-Pad1)
- C8 pad 2: +BATT -> GNDPWR
- C9 pad 1: Net-(C9-Pad1) -> GNDPWR
- C9 pad 2: GNDPWR -> +BATT
- DA1 pad 1: Net-(D1-PadA) -> Net-(C10-Pad1)
- DA1 pad 10: Net-(C10-Pad2) -> /L1IN
- DA1 pad 2: Net-(DA1-Pad2) -> +BATT
- DA1 pad 3: Net-(C9-Pad1) -> (no net)
- DA1 pad 4: +BATT -> Net-(C23-Pad1)
- DA1 pad 5: Net-(C11-Pad2) -> GNDPWR
- DA1 pad 6: Net-(DA1-Pad6) -> Net-(C8-Pad1)
- DA1 pad 7: GNDPWR -> Net-(DA1-Pad7)
- DA1 pad 8: Net-(C10-Pad1) -> Net-(DA1-Pad8)
- DA1 pad 9: Net-(DA1-Pad9) -> GNDPWR
- L1 pad 2: Net-(C10-Pad1) -> /L1IN
- Q1 pad 1: Net-(C10-Pad1) -> /L1IN
- Q1 pad 2: Net-(DA1-Pad9) -> /L1IN
- Q1 pad 3: GNDPWR -> /L1IN
- Q1 pad 4: Net-(DA1-Pad6) -> Net-(DA1-Pad11)
- Q1 pad 5: Net-(C10-Pad1) -> +BATT
- Q1 pad 6: Net-(C10-Pad1) -> +BATT
- R1 pad 1: /SHLD -> Net-(DA1-Pad7)
- R1 pad 2: GND -> +BATT
- R2 pad 1: Net-(D1-PadA) -> /L1IN
- R2 pad 2: Net-(C6-Pad2) -> Net-(DA1-Pad8)
- R3 pad 1: Net-(C11-Pad2) -> Net-(C23-Pad1)
- R3 pad 2: Net-(C9-Pad1) -> +5V
- R4 pad 2: Net-(DA1-Pad2) -> Net-(C23-Pad1)
- R5 pad 1: +5V -> +3.3V
- R5 pad 2: Net-(DA1-Pad2) -> Net-(C26-Pad2)
Routing:
- net Net-(C10-Pad1): track 30.3 -> 0.52 mm
- net /L1IN: track 0.00 -> 27.8 mm, vias 0 -> 2
- net /SHLD: track 27.3 -> 0.00 mm, vias 2 -> 0
- net GNDPWR: track 277.5 -> 252.2 mm, vias 14 -> 11
- net VCC: track 58.9 -> 42.5 mm, vias 6 -> 5
- net +BATT: track 122.7 -> 138.5 mm, vias 1 -> 5
- net Net-(DA1-Pad6): track 12.5 -> 0.00 mm, vias 2 -> 0
- net Net-(DA1-Pad9): track 11.4 -> 0.00 mm, vias 2 -> 0
- net Net-(C23-Pad1): track 0.00 -> 11.1 mm, vias 0 -> 2
- net GND: track 399.6 -> 390.4 mm, vias 92 -> 90
- net (no net): track 0.00 -> 9.19 mm, vias 0 -> 2
- net Net-(C9-Pad1): track 8.69 -> 0.00 mm, vias 2 -> 0
- net Net-(DA1-Pad2): track 5.74 -> 0.00 mm
- net Net-(DA1-Pad11): track 0.00 -> 5.48 mm
- net Net-(C10-Pad2): track 5.36 -> 0.00 mm
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
Commit message: v2 sent to factory
Parts:
- BLN1: value BALUN868ST -> BALUN868JOHANSON; footprint Radio:BALUN868_ST -> Radio:BALUN_JOHANSON868
- moved R15 84.7 mm to (151.8, 112.2)
- moved C47 77.6 mm to (123.0, 90.2), turned to 180 degrees
- moved C46 76.3 mm to (128.4, 93.8), turned to 270 degrees
- moved XL3 75.6 mm to (166.4, 92.2), turned to 180 degrees
- moved DA7 73.7 mm to (157.6, 110.4), turned to 270 degrees
- moved Q2 71.1 mm to (145.5, 116.0), turned to 270 degrees
- moved C45 70.9 mm to (133.1, 88.7)
- moved C44 62.4 mm to (131.4, 84.6)
- moved C1 47.5 mm to (128.0, 124.4)
- moved R1 45.3 mm to (132.0, 124.0)
- moved C21 44.7 mm to (162.4, 107.6), turned to 90 degrees
- moved C18 39.9 mm to (165.8, 105.2), turned to 180 degrees
- moved C26 31.6 mm to (151.2, 109.4), turned to 270 degrees
- moved C23 28.8 mm to (129.4, 112.2)
- moved R5 23.7 mm to (152.8, 109.4), turned to 270 degrees
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Routing:
- net +BATT: track 138.5 -> 233.7 mm, vias 5 -> 0
- net GNDPWR: track 252.2 -> 343.1 mm, vias 11 -> 39
- net /ANT2: track 13.5 -> 56.7 mm
- net /L1IN: track 27.8 -> 63.1 mm, vias 2 -> 3
- net +5V: track 140.1 -> 119.4 mm, vias 38 -> 29
- net GND: track 390.4 -> 373.3 mm, vias 90 -> 60
- net VCC: track 42.5 -> 57.4 mm, vias 5 -> 7
- net Net-(C26-Pad2): track 1.57 -> 14.5 mm
- net +3.3V: track 30.2 -> 39.5 mm, vias 0 -> 2
- net (no net): track 9.19 -> 0.00 mm, vias 2 -> 0
- net Net-(DA1-Pad11): track 5.48 -> 14.6 mm, vias 0 -> 2
- net Net-(DA1-Pad8): track 2.11 -> 10.2 mm, vias 0 -> 2
- net PwrMCU: track 61.4 -> 68.0 mm, vias 6 -> 4
- net Net-(DD1-Pad42): track 15.2 -> 20.7 mm
- net /5V_USB: track 16.2 -> 21.3 mm, vias 4 -> 3
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Other:
- board text added: "12V Ctrl"
- board text added: "LedBandRadio v2"
- board text removed: "LedBandRadio v1"
