File: LedBandRadio_hw/LedBandRadio.sch (KiCad schematic (older format))
At the start: 99 parts, among them Q1 IRF8313, SW1 DIPx6, U1 USBLC6

Commit message: New +5V sch Still with 3-ch 12V LED control
Parts:
- removed D1, D2: BAT54WS, Diodes:SOD323, symbol D_Shottky
- removed DA1: MAX8546, SO_DIL_TSSOP:uMAX_uSOP10, symbol MAX8546
- removed Q1: IRF8313, SO_DIL_TSSOP:SO8_150MIL, symbol Nx2_SO8
- added C44, C45, C46, C47: 0.1u, Capacitors:CAP_0603, symbol C
- added DA1: LM3150, SO_DIL_TSSOP:HTSSOP14, symbol LM3150
- added DA7: LP2951, SO_DIL_TSSOP:SO8_150MIL, symbol LP2951
- added Q1, Q2: IRF8714, SO_DIL_TSSOP:SO8_150MIL, symbol N_SO8
- added R15: 10k, Resistors:RES_0603, symbol R
- C1, C6: value 10n -> 10u 16V; footprint Capacitors:CAP_0603 -> Capacitors:CAP_0805; PN (none) -> CL21A106KOQNNNE; Price 0.5 -> 1.6; URL (none) -> http://onelec.ru/products/cl21a106koqnnne-dfe76b50-f77a-465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
- C10: value 0.22u -> 1u
- C11: value 1u -> 0.47u
- C21, C34: value 220pF -> 0.1u
- C23: value 10n -> 470pF; PN (none) -> CC0603JRNPO9BN471; Price (none) -> 0.5; SolderPoints (none) -> 2; URL (none) -> http://onelec.ru/products/cc0603jrnpo9bn471-6aeb18ba-053d-4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
- C26: value 3.3pF -> 10n
- C28: value 10n -> 1u
- C8: value 1u -> 0.1u
- F7: footprint Resistors:RES_0603_FUSE -> PCB:FuseShorted
- L1: footprint Inductors:13x14 -> Inductors:13x13
- R1: value 1M -> 100k
- R2: value 47k -> 2k
- R3: value 10R -> 75k
- R4: value 4.7k -> 10k
- R5: value 27k -> 12k; Price 0.5 -> (none); SolderPoints 2 -> (none)
- R6: value 220R -> 1k
Connections:
- net labels added: L1IN
- net labels removed: SHLD
- wire segments 327 -> 360
- no-connect marks 12 -> 20
Other:
- note added: "2.7V if powerful 5V not required"
- note added: "2k => ILim=9.5A"
- note added: "5V 10A"
- note added: "75k + 10k => 5.1V"
- note added: "Power input"
- note added: "Soft Start:\n100n => 7.8mS"
- note removed: "Locket case:\nC23 = ???\nC25 - ???\nL4 = ???"

Commit message: v2 sent to factory
Parts:
- removed BLN1: BALUN868ST, Radio:BALUN868_ST, symbol BALUN868ST
- added BLN1: BALUN868JOHANSON, Radio:BALUN_JOHANSON868, symbol BALUN868JOHANSON
Connections:
- wire segments 360 -> 363

Commit message: Antenna matched on the desk
Parts:
- removed C41: *, Capacitors:CAP_0402, symbol C
- added C?: 100pF, Capacitors:CAP_0402, symbol C
- added C?: 1.5pF, Capacitors:CAP_0402, symbol C
- C42: value * -> DoNotMount
- L4: value * -> 5.6nH
Connections:
- wire segments 363 -> 364
Other:
- note added: "Add it\nsomehow"
Changed lines of the file:
@@
 L GND #PWR92
 U 1 1 57197DE2
-P 13400 2700
-F 0 "#PWR92" H 13490 2680 30  0001 C CNN
-F 1 "GND" H 13400 2620 30  0001 C CNN
-F 2 "" H 13400 2700 60  0001 C CNN
-F 3 "" H 13400 2700 60  0001 C CNN
-	1    13400 2700
-	1    0    0    -1
-$EndComp
-Text Notes 13400 1600 0    60   ~ 0
+P 13950 2700
+F 0 "#PWR92" H 14040 2680 30  0001 C CNN
+F 1 "GND" H 13950 2620 30  0001 C CNN
+F 2 "" H 13950 2700 60  0001 C CNN
+F 3 "" H 13950 2700 60  0001 C CNN
+	1    13950 2700
+	1    0    0    -1
+$EndComp
+Text Notes 13950 1600 0    60   ~ 0
 Matching circuit
 $Comp
@@
 	1    0    0    -1
 $EndComp
-Text Label 13350 1950 0    60   ~ 0
+Text Label 13900 1950 0    60   ~ 0
 ANT1
 Entry Wire Line
@@
 L GND #PWR93
 U 1 1 57197DF7
-P 14100 2700
-F 0 "#PWR93" H 14190 2680 30  0001 C CNN
-F 1 "GND" H 14100 2620 30  0001 C CNN
-F 2 "" H 14100 2700 60  0001 C CNN
-F 3 "" H 14100 2700 60  0001 C CNN
-	1    14100 2700
+P 14650 2700
+F 0 "#PWR93" H 14740 2680 30  0001 C CNN
+F 1 "GND" H 14650 2620 30  0001 C CNN
+F 2 "" H 14650 2700 60  0001 C CNN
+F 3 "" H 14650 2700 60  0001 C CNN
+	1    14650 2700
 	1    0    0    -1
 $EndComp
 Text Notes 12600 1550 0    60   ~ 0
 Balun
-Text Label 14150 1950 0    60   ~ 0
+Text Label 14700 1950 0    60   ~ 0
 ANT2
 Text Label 9750 1900 2    60   ~ 0
@@
 L L L4
 U 1 1 57197E49
-P 13750 1950
-F 0 "L4" V 13650 1810 40  0000 C CNN
-F 1 "*" V 13650 1950 40  0000 C CNN
-F 2 "Inductors:IND_0402" V 13810 1960 40  0001 C CNN
-F 3 "" V 13650 1810 60  0001 C CNN
-F 4 "4" V 13750 1910 60  0001 C CNN "Price"
-F 5 "2" V 13850 2010 60  0001 C CNN "SolderPoints"
-	1    13750 1950
-	0    1    1    0
-$EndComp
-$Comp
-L C C41
-U 1 1 57197E52
-P 13400 2450
-F 0 "C41" H 13300 2350 50  0000 L CNN
-F 1 "*" H 13300 2550 50  0000 L CNN
-F 2 "Capacitors:CAP_0402" V 13500 2300 28  0001 C BNN
-F 3 "" H 13300 2350 60  0001 C CNN
-F 4 "0.5" H 13400 2450 60  0001 C CNN "Price"
-F 5 "2" H 13500 2550 60  0001 C CNN "SolderPoints"
-	1    13400 2450
+P 13950 2450
+F 0 "L4" V 13850 2310 40  0000 C CNN
+F 1 "5.6nH" V 13850 2450 40  0000 C CNN
+F 2 "Inductors:IND_0402" V 14010 2460 40  0001 C CNN
+F 3 "" V 13850 2310 60  0001 C CNN
+F 4 "4" V 13950 2410 60  0001 C CNN "Price"
+F 5 "2" V 14050 2510 60  0001 C CNN "SolderPoints"
+	1    13950 2450
 	1    0    0    -1
 $EndComp
@@
 L C C42
 U 1 1 57197E5B
-P 14100 2450
-F 0 "C42" H 14000 2350 50  0000 L CNN
-F 1 "*" H 14000 2550 50  0000 L CNN
-F 2 "Capacitors:CAP_0402" V 14200 2300 28  0001 C BNN
-F 3 "" H 14000 2350 60  0001 C CNN
-F 4 "0.5" H 14100 2450 60  0001 C CNN "Price"
-F 5 "2" H 14200 2550 60  0001 C CNN "SolderPoints"
-	1    14100 2450
+P 14650 2450
+F 0 "C42" H 14550 2350 50  0000 L CNN
+F 1 "DoNotMount" H 14550 2550 50  0000 L CNN
+F 2 "Capacitors:CAP_0402" V 14750 2300 28  0001 C BNN
+F 3 "" H 14550 2350 60  0001 C CNN
+F 4 "0.5" H 14650 2450 60  0001 C CNN "Price"
+F 5 "2" H 14750 2550 60  0001 C CNN "SolderPoints"
+	1    14650 2450
 	1    0    0    -1
 $EndComp
@@
 	11900 1950 12250 1950
 Wire Wire Line
-	13150 1950 13550 1950
-Connection ~ 13400 1950
-Wire Wire Line
-	14100 2650 14100 2700
-Wire Wire Line
-	14100 1950 14100 2250
+	13700 1950 14100 1950
+Connection ~ 13950 1950
+Wire Wire Line
+	14650 2650 14650 2700
+Wire Wire Line
+	14650 1950 14650 2250
 Wire Bus Line
 	9900 1450 9900 2550
 Wire Wire Line
 	10000 2450 10550 2450
-Connection ~ 14100 1950
-Wire Wire Line
-	13950 1950 14500 1950
+Connection ~ 14650 1950
+Wire Wire Line
+	14500 1950 15050 1950
 Wire Wire Line
 	12800 2400 12800 2600
 Wire Wire Line
-	13400 2650 13400 2700
-Wire Wire Line
-	13400 1950 13400 2250
+	13950 2650 13950 2700
+Wire Wire Line
+	13950 1950 13950 2250
 Wire Wire Line
 	9850 3200 9950 3200
@@
 L ANT_GENERAL ANT1
 U 1 1 57316822
-P 14950 2000
-F 0 "ANT1" H 14650 2250 60  0000 C CNN
-F 1 "ANT_GENERAL" H 14850 2150 60  0000 C CNN
-F 2 "Radio:ANT_INVF_LEDBANDRXTX" H 14950 2000 60  0001 C CNN
-F 3 "" H 14950 2000 60  0000 C CNN
-	1    14950 2000
+P 15500 2000
+F 0 "ANT1" H 15200 2250 60  0000 C CNN
+F 1 "ANT_GENERAL" H 15400 2150 60  0000 C CNN
+F 2 "Radio:ANT_INVF_LEDBANDRXTX" H 15500 2000 60  0001 C CNN
+F 3 "" H 15500 2000 60  0000 C CNN
+	1    15500 2000
 	1    0    0    -1
 $EndComp
@@
 L GND #PWR94
 U 1 1 57317055
-P 14500 2100
-F 0 "#PWR94" H 14590 2080 30  0001 C CNN
-F 1 "GND" H 14500 2020 30  0001 C CNN
-F 2 "" H 14500 2100 60  0001 C CNN
-F 3 "" H 14500 2100 60  0001 C CNN
-	1    14500 2100
-	1    0    0    -1
-$EndComp
-Wire Wire Line
-	14500 2050 14500 2100
+P 15050 2100
+F 0 "#PWR94" H 15140 2080 30  0001 C CNN
+F 1 "GND" H 15050 2020 30  0001 C CNN
+F 2 "" H 15050 2100 60  0001 C CNN
+F 3 "" H 15050 2100 60  0001 C CNN
+	1    15050 2100
+	1    0    0    -1
+$EndComp
+Wire Wire Line
+	15050 2050 15050 2100
 $Comp
 L Fuse0R F7
@@
 Wire Wire Line
 	12900 2500 12900 2400
+$Comp
+L C C?
+U 1 1 597525FC
+P 13500 1950
+F 0 "C?" V 13400 1800 50  0000 L CNN
+F 1 "100pF" V 13400 2050 50  0000 L CNN
+F 2 "Capacitors:CAP_0402" V 13600 1800 28  0001 C BNN
+F 3 "" H 13400 1850 60  0001 C CNN
+F 4 "0.5" H 13500 1950 60  0001 C CNN "Price"
+F 5 "2" H 13600 2050 60  0001 C CNN "SolderPoints"
+	1    13500 1950
+	0    1    1    0
+$EndComp
+Wire Wire Line
+	13300 1950 13150 1950
+Text Notes 13300 1800 0    60   ~ 0
+Add it\nsomehow
+$Comp
+L C C?
+U 1 1 59753680
+P 14300 1950
+F 0 "C?" V 14200 1800 50  0000 L CNN
+F 1 "1.5pF" V 14200 2050 50  0000 L CNN
+F 2 "Capacitors:CAP_0402" V 14400 1800 28  0001 C BNN
+F 3 "" H 14200 1850 60  0001 C CNN
+F 4 "0.5" H 14300 1950 60  0001 C CNN "Price"
+F 5 "2" H 14400 2050 60  0001 C CNN "SolderPoints"
+	1    14300 1950
+	0    1    1    0
+$EndComp
 $EndSCHEMATC

Commit message: * sch
Parts:
- ANT1: symbol ANT_GENERAL -> Antennas_kl:ANT_GENERAL
- BLN1: symbol BALUN868JOHANSON -> RFICs:BALUN868JOHANSON
- C1, C10, C11, C12, C15, C17, C18, C19, C2, C20, C21, C22, C23, C24, C25, C26, C27, C28, C29, C30, C31, C32, C33, C34, C35, C36, C37, C38, C39, C4, C40, C42, C43, C44, C45, C46, C47, C6, C8, C9, C? (x2): symbol C -> Tittar_kl:C
- C13, C14, C16, C3, C5, C7: symbol CP -> Tittar_kl:CP
- D3, D4: symbol D_Shottky -> Tittar_kl:D_Shottky
- D5: symbol LED -> Tittar_kl:LED
- DA1: symbol LM3150 -> Power_kl:LM3150
- DA2: symbol NCP583SQ -> Power_kl:NCP583SQ
- DA3: symbol MC74VHC1 -> standard_logic:MC74VHC1
- DA4, DA5, DA6: symbol IPS6041 -> Power_kl:IPS6041
- DA7: symbol LP2951 -> Power_kl:LP2951
- DD1: symbol STM32L151CxTx -> st_kl:STM32L151CxTx
- DD2: symbol CC1101 -> RFICs:CC1101
- F1, F2, F3, F4, F5, F6, F7: symbol Fuse0R -> Tittar_kl:Fuse0R
- HOLE1, HOLE2: symbol HOLE_METALLED -> pcb_details:HOLE_METALLED
- L1, L2, L3, L4: symbol L -> Tittar_kl:L
- Logo1: symbol Logo -> pcb_details:Logo
- Q1, Q2: symbol N_SO8 -> Transistors_kl:N_SO8
- R1, R10, R11, R12, R13, R14, R15, R2, R3, R4, R5, R6, R7, R8, R9: symbol R -> Tittar_kl:R
- SW1: symbol DIPx6 -> Switches:DIPx6
- TP1, TP2: symbol TESTPOINT -> pcb_details:TESTPOINT
- U1: symbol USBLC6 -> ESDProtection:USBLC6
- XL1: symbol CONN_6 -> Connectors_kl:CONN_6
- XL2: symbol CONN_2 -> Connectors_kl:CONN_2
- XL3: symbol USB_MINI_B -> Connectors_kl:USB_MINI_B
- XL4: symbol CONN_5 -> Connectors_kl:CONN_5
- XL5: symbol CONN_3 -> Connectors_kl:CONN_3
- XL6: symbol CONN_4 -> Connectors_kl:CONN_4
- XTAL1, XTAL2: symbol CRYSTAL_H -> Tittar_kl:CRYSTAL_H
Connections:
- wire segments 364 -> 482

Commit message: RC
Parts:
- DA3: symbol standard_logic:MC74VHC1 -> standard_logic:1xBUF_W3STATE
- gave numbers to parts that had none: 2
Connections:
- net labels added: +3v3, +5v
- net labels removed: +3.3V, +5V
Other:
- moved on the sheet: D3, D4
